File: Hardware/ADC shield V2.0/IotaWatt.brd (EAGLE design)
At the start: 53.6 x 61 mm, 58 parts, among them J0 STEREO_JACK_BOT, J1 STEREO_JACK_BOT, J2 STEREO_JACK_BOT, J3 STEREO_JACK_BOT, J4 STEREO_JACK_BOT, J5 STEREO_JACK_BOT, J6 STEREO_JACK_BOT

Commit message: Fix connection
Routing:
- net N$2: track 29.3 -> 36.2 mm, vias 0 -> 2
Changed lines of the file:
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@@
 <grid distance="0.025" unitdist="inch" unit="inch" style="dots" multiple="2" display="yes" altdistance="0.00625" altunitdist="inch" altunit="inch"/>
 <layers>
-<layer number="1" name="Top" color="4" fill="1" visible="yes" active="yes"/>
+<layer number="1" name="Top" color="59" fill="1" visible="yes" active="yes"/>
 <layer number="16" name="Bottom" color="1" fill="1" visible="yes" active="yes"/>
 <layer number="17" name="Pads" color="2" fill="1" visible="yes" active="yes"/>
@@
 <layer number="105" name="Beschreib" color="9" fill="1" visible="yes" active="yes"/>
 <layer number="106" name="BGA-Top" color="4" fill="1" visible="yes" active="yes"/>
-<layer number="107" name="BD-Top" color="5" fill="1" visible="yes" active="yes"/>
+<layer number="107" name="BD-Top" color="59" fill="1" visible="yes" active="yes"/>
 <layer number="108" name="fp8" color="7" fill="1" visible="yes" active="yes"/>
 <layer number="109" name="fp9" color="7" fill="1" visible="yes" active="yes"/>
@@
 <wire x1="2.175" y1="31.59125" x2="2.7" y2="34.19" width="0.254" layer="1"/>
 <wire x1="2.7" y1="34.19" x2="2.175" y2="36.83" width="0.254" layer="1"/>
-<wire x1="2.8" y1="34.29" x2="2.7" y2="34.19" width="0.254" layer="1" curve="90"/>
-<wire x1="5.715" y1="34.29" x2="5.715" y2="41.275" width="0.254" layer="1"/>
-<wire x1="5.715" y1="34.29" x2="5.715" y2="33.655" width="0.254" layer="1"/>
-<wire x1="5.715" y1="33.655" x2="7.58" y2="31.79" width="0.254" layer="1" curve="90"/>
-<wire x1="7.7" y1="31.79" x2="7.58" y2="31.79" width="0.254" layer="1"/>
-<wire x1="2.7" y1="34.19" x2="5.715" y2="34.29" width="0.254" layer="1"/>
+<wire x1="2.7" y1="34.19" x2="2.8" y2="34.29" width="0.254" layer="1" curve="-90"/>
+<wire x1="7.58" y1="31.79" x2="7.7" y2="31.79" width="0.254" layer="1"/>
 <wire x1="10.16" y1="29.63" x2="13.0175" y2="29.0195" width="0.254" layer="1"/>
 <wire x1="10.16" y1="29.63" x2="7.7" y2="29.09" width="0.254" layer="1"/>
 <wire x1="7.7" y1="29.09" x2="7.7" y2="31.79" width="0.254" layer="1"/>
 <wire x1="11.43" y1="46.14875" x2="11.43" y2="43.8625" width="0.254" layer="1"/>
-<wire x1="5.715" y1="41.275" x2="11.43" y2="43.8625" width="0" layer="19" extent="1-1"/>
+<via x="9.525" y="43.815" extent="1-16" drill="0.6"/>
+<wire x1="9.525" y1="43.815" x2="11.43" y2="43.815" width="0.254" layer="1"/>
+<via x="9.525" y="33.655" extent="1-16" drill="0.6"/>
+<wire x1="9.525" y1="33.655" x2="9.525" y2="43.815" width="0.254" layer="16"/>
+<wire x1="2.8" y1="34.29" x2="7.7" y2="31.79" width="0.254" layer="1"/>
+<wire x1="7.7" y1="31.79" x2="9.525" y2="33.655" width="0.254" layer="1"/>
+<wire x1="11.43" y1="43.815" x2="11.43" y2="43.8625" width="0" layer="19" extent="1-1"/>
 </signal>
 <signal name="GND">
@@
 <via x="43.18" y="46.99" extent="1-16" drill="0.6"/>
 <via x="10.16" y="21.59" extent="1-16" drill="0.6"/>
-<via x="10.16" y="34.29" extent="1-16" drill="0.6"/>
+<via x="11.1125" y="33.3375" extent="1-16" drill="0.6"/>
 <via x="10.16" y="8.89" extent="1-16" drill="0.6"/>
 <via x="4.445" y="15.08125" extent="1-16" drill="0.6"/>
