File: Hardware/IotaWatt4.3.sch (EAGLE design)
At the start: 59 parts, among them J0 2.1MMJACKSMT, J1 STEREO_SMD, J10 STEREO_SMD, J11 STEREO_SMD, J12 STEREO_SMD, J13 STEREO_SMD, J14 STEREO_SMD, J2 STEREO_SMD, J3 STEREO_SMD, J4 STEREO_SMD, J5 STEREO_SMD, J6 STEREO_SMD, J7 STEREO_SMD, J8 STEREO_SMD, J9 STEREO_SMD, Y1 32Khz

Commit message: Update version and date
Other:
- note added: "IotaWatt Electric Power Monitor Version 4.3 August 14, 2017"
- note removed: "IotaWatt Electric Power Monitor Version 4.1 July 6, 2017"
Changed lines of the file:
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@@
 <text x="190.5" y="-101.6" size="5.08" layer="91">IotaWatt
 Electric Power Monitor
-Version 4.1
-July 6, 2017</text>
+Version 4.3
+August 14, 2017</text>
 <text x="190.5" y="76.2" size="1.778" layer="91">alternate location</text>
 <text x="164.338" y="-24.384" size="2.54" layer="91">LM358</text>
